Commit message: Refactor - rename projects.

File: acky_bot_description/urdf/bicycle.urdf.xacro (robot description, xacro)
@@ -2,7 +2,7 @@
 <robot xmlns:xacro="http://www.ros.org/wiki/xacro" name="bicycle">
     <!-- Xacro includes -->
-    <xacro:include filename="$(find ursa_bot_description)/urdf/materials.xacro"/>
-    <xacro:include filename="$(find ursa_bot_description)/urdf/inertials.xacro"/>
-    <xacro:property name="robot_namespace" value="/ursa_bot"/>
+    <xacro:include filename="$(find acky_bot_description)/urdf/materials.xacro"/>
+    <xacro:include filename="$(find acky_bot_description)/urdf/inertials.xacro"/>
+    <xacro:property name="robot_namespace" value="/acky_bot"/>
     <!-- Gazebo plugins -->
     <gazebo>

File: acky_bot_description/urdf/ursa_bot.urdf.xacro (robot description, xacro)
@@ -1,5 +1,5 @@
 <?xml version="1.0"?>
-<robot xmlns:xacro="http://www.ros.org/wiki/xacro" name="ursa_bot">
-    <xacro:include filename="$(find ursa_bot_description)/urdf/inertials.xacro"/>
+<robot xmlns:xacro="http://www.ros.org/wiki/xacro" name="acky_bot">
+    <xacro:include filename="$(find acky_bot_description)/urdf/inertials.xacro"/>
     <!-- Degree-to-radian conversions -->
     <xacro:property name="degrees_45" value="0.785398163"/>

Commit message: Simplify geometry for bicycle model.

File: acky_bot_description/urdf/bicycle.urdf.xacro (robot description, xacro)
@@ -28,20 +28,20 @@
     <xacro:property name="degrees_180" value="3.14159265"/>
     <!-- Basic Geometry of Body -->
-    <xacro:property name="body_length" value="1.91" />
-    <xacro:property name="body_width" value="0.680618" />
-    <xacro:property name="body_height" value="1.065022" />
-    <xacro:property name="body_mass" value="20"/>
+    <xacro:property name="body_length" value="2.0" />
+    <xacro:property name="body_width" value="0.7" />
+    <xacro:property name="body_height" value="1.0" />
+    <xacro:property name="body_mass" value="10"/>
     <!-- Front Steer (Motor) Properties -->
     <xacro:property name="front_steer_width" value="0.4" />
     <xacro:property name="front_steer_diameter" value="0.3" />
-    <xacro:property name="front_steer_mass" value="10"/>
+    <xacro:property name="front_steer_mass" value="2"/>
     <!-- Front Wheel Properties -->
     <xacro:property name="front_wheel_width" value="0.4" />
     <xacro:property name="front_wheel_diameter" value="0.6" />
-    <xacro:property name="front_wheel_mass" value="20"/>
+    <xacro:property name="front_wheel_mass" value="5"/>
     <!-- Rear Wheel Properties -->
     <xacro:property name="rear_wheel_width" value="0.4" />
     <xacro:property name="rear_wheel_diameter" value="0.6" />
-    <xacro:property name="rear_wheel_mass" value="20"/>
+    <xacro:property name="rear_wheel_mass" value="5"/>
     <!-- Base Link -->
     <link name="base_link">

File: acky_bot_description/urdf/inertials.xacro (robot description, xacro)
@@ -1,33 +1,4 @@
 <?xml version="1.0" ?>
-<!--
-    Software License Agreement (BSD-3-Clause)
-    Copyright (c) 2019 Rhys Mainwaring
-    All rights reserved.
-    Redistribution and use in source and binary forms, with or without
-    modification, are permitted provided that the following conditions
-    are met:
-    1.  Redistributions of source code must retain the above copyright
-        notice, this list of conditions and the following disclaimer.
-    2.  Redistributions in binary form must reproduce the above
-        copyright notice, this list of conditions and the following
-        disclaimer in the documentation and/or other materials provided
-        with the distribution.
-    3.  Neither the name of the copyright holder nor the names of its
-        contributors may be used to endorse or promote products derived
-        from this software without specific prior written permission.
-    THIS SOFTWARE IS PROVIDED BY THE COPYRIGHT HOLDERS AND CONTRIBUTORS
-    "AS IS" AND ANY EXPRESS OR IMPLIED WARRANTIES, INCLUDING, BUT NOT
-    LIMITED TO, THE IMPLIED WARRANTIES OF MERCHANTABILITY AND FITNESS
-    FOR A PARTICULAR PURPOSE ARE DISCLAIMED. IN NO EVENT SHALL THE
-    COPYRIGHT HOLDER OR CONTRIBUTORS BE LIABLE FOR ANY DIRECT, INDIRECT,
-    INCIDENTAL, SPECIAL, EXEMPLARY, OR CONSEQUENTIAL DAMAGES (INCLUDING,
-    BUT NOT LIMITED TO, PROCUREMENT OF SUBSTITUTE GOODS OR SERVICES;
-    LOSS OF USE, DATA, OR PROFITS; OR BUSINESS INTERRUPTION) HOWEVER
-    CAUSED AND ON ANY THEORY OF LIABILITY, WHETHER IN CONTRACT, STRICT
-    LIABILITY, OR TORT (INCLUDING NEGLIGENCE OR OTHERWISE) ARISING IN
-    ANY WAY OUT OF THE USE OF THIS SOFTWARE, EVEN IF ADVISED OF THE
-    POSSIBILITY OF SUCH DAMAGE.
--->
-<!--  xacro macros for intertials.
+<!--  xacro macros for inertials.
     Define xacro macros for math constants and inertials:
     - solid cuboid

File: acky_bot_description/urdf/materials.xacro (robot description, xacro)
@@ -1,32 +1,3 @@
 <?xml version="1.0" ?>
-<!--
-    Software License Agreement (BSD-3-Clause)
-    Copyright (c) 2019 Rhys Mainwaring
-    All rights reserved.
-    Redistribution and use in source and binary forms, with or without
-    modification, are permitted provided that the following conditions
-    are met:
-    1.  Redistributions of source code must retain the above copyright
-        notice, this list of conditions and the following disclaimer.
-    2.  Redistributions in binary form must reproduce the above
-        copyright notice, this list of conditions and the following
-        disclaimer in the documentation and/or other materials provided
-        with the distribution.
-    3.  Neither the name of the copyright holder nor the names of its
-        contributors may be used to endorse or promote products derived
-        from this software without specific prior written permission.
-    THIS SOFTWARE IS PROVIDED BY THE COPYRIGHT HOLDERS AND CONTRIBUTORS
-    "AS IS" AND ANY EXPRESS OR IMPLIED WARRANTIES, INCLUDING, BUT NOT
-    LIMITED TO, THE IMPLIED WARRANTIES OF MERCHANTABILITY AND FITNESS
-    FOR A PARTICULAR PURPOSE ARE DISCLAIMED. IN NO EVENT SHALL THE
-    COPYRIGHT HOLDER OR CONTRIBUTORS BE LIABLE FOR ANY DIRECT, INDIRECT,
-    INCIDENTAL, SPECIAL, EXEMPLARY, OR CONSEQUENTIAL DAMAGES (INCLUDING,
-    BUT NOT LIMITED TO, PROCUREMENT OF SUBSTITUTE GOODS OR SERVICES;
-    LOSS OF USE, DATA, OR PROFITS; OR BUSINESS INTERRUPTION) HOWEVER
-    CAUSED AND ON ANY THEORY OF LIABILITY, WHETHER IN CONTRACT, STRICT
-    LIABILITY, OR TORT (INCLUDING NEGLIGENCE OR OTHERWISE) ARISING IN
-    ANY WAY OUT OF THE USE OF THIS SOFTWARE, EVEN IF ADVISED OF THE
-    POSSIBILITY OF SUCH DAMAGE.
--->
 <!--  xacro macros for robot materials.
  -->
