Commit message: Add steer_bot model from https://github.com/CIR-KIT/steer_drive_ros/blob/kinetic-devel/steer_drive_controller/test/common/urdf/steerbot.xacro
1. Add steer_bot model and update transmission elements, inertials and parameter definitions
2. Add rviz launch file for steer_bot
3. Move other models into separate folders.

File: acky_bot_description/urdf/bicycle_bot/bicycle_bot.urdf.xacro (robot description, xacro)
@@ -1,7 +1,7 @@
 <?xml version="1.0"?>
-<robot xmlns:xacro="http://www.ros.org/wiki/xacro" name="bicycle">
-    <!-- Xacro includes -->
-    <xacro:include filename="$(find acky_bot_description)/urdf/materials.xacro"/>
-    <xacro:include filename="$(find acky_bot_description)/urdf/inertials.xacro"/>
+<robot  name="bicycle_bot" xmlns:xacro="http://wiki.ros.org/xacro">
+    <!-- xacro includes -->
+    <xacro:include filename="$(find acky_bot_description)/urdf/common/materials.xacro"/>
+    <xacro:include filename="$(find acky_bot_description)/urdf/common/inertials.xacro"/>
     <xacro:property name="robot_namespace" value="/acky_bot"/>
     <!-- Gazebo plugins -->

File: acky_bot_description/urdf/common/inertials.xacro (robot description, xacro)
@@ -6,5 +6,5 @@
     - null (a placeholder inertial for logical link elements)
  -->
-<robot name="inertials" xmlns:xacro="http://www.ros.org/wiki/xacro">
+<robot name="inertials" xmlns:xacro="http://wiki.ros.org/xacro">
     <!-- Math constants -->
     <xacro:property name="math_pi"        value="3.141592653589793" />

File: acky_bot_description/urdf/common/materials.xacro (robot description, xacro)
@@ -2,5 +2,5 @@
 <!--  xacro macros for robot materials.
  -->
-<robot name="materials" xmlns:xacro="http://www.ros.org/wiki/xacro">
+<robot name="materials" xmlns:xacro="http://wiki.ros.org/xacro">
    <material name="red">
         <color rgba="0.8 0 0 1"/>
@@ -11,4 +11,7 @@
     <material name="blue">
         <color rgba="0 0 0.8 1"/>
+    </material>
+    <material name="yellow">
+        <color rgba="0.8 0.8 0 1"/>
     </material>
     <material name="orange">

File: acky_bot_description/urdf/ursa_bot/ursa_bot.urdf.xacro (robot description, xacro)
@@ -1,16 +1,20 @@
 <?xml version="1.0"?>
 <robot xmlns:xacro="http://www.ros.org/wiki/xacro" name="acky_bot">
+    <!-- xacro includes -->
     <xacro:include filename="$(find acky_bot_description)/urdf/inertials.xacro"/>
+    <xacro:property name="robot_namespace" value="/acky_bot"/>
+    <!-- Gazebo plugin for ROS Control
+        See: http://wiki.ros.org/steer_bot_hardware_gazebo?distro=indigo
+    -->
+    <gazebo>
+        <plugin name="gazebo_ros_control" filename="libgazebo_ros_control.so">
+            <robotNamespace>${robot_namespace}</robotNamespace>
+            <robotSimType>steer_bot_hardware_gazebo/SteerBotHardwareGazebo</robotSimType>
+        </plugin>
+    </gazebo>
     <!-- Degree-to-radian conversions -->
     <xacro:property name="degrees_45" value="0.785398163"/>
     <xacro:property name="degrees_90" value="1.57079633"/>
     <xacro:property name="degrees_180" value="3.14159265"/>
-    <!-- Inertia Generator -->
-    <xacro:macro name="default_inertial" params="mass">
-        <inertial>
-            <mass value="${mass}" />
-            <inertia ixx="1.5" ixy="0.0" ixz="0.0" iyy="1.5" iyz="0.0" izz="1.5" />
-        </inertial>
-    </xacro:macro>
     <!-- Basic Geometry of Body -->
     <xacro:property name="body_length" value="1.91" />
@@ -52,5 +56,5 @@
         <link name="${prefix}_steering_link">
             <visual>
-                <origin xyz="0.0 0.0 0.0" rpy="${degrees_90} 0.0 0.0"/>
+                <origin xyz="0 0 0" rpy="${degrees_90} 0 0"/>
                 <geometry>
                     <cylinder radius="${steering_diameter}" length="${steering_width}"/>
@@ -58,10 +62,13 @@
             </visual>
             <collision>
-                <origin xyz="0.0 0.0 0.0" rpy="${degrees_90} 0.0 0.0"/>
+                <origin xyz="0 0 0" rpy="${degrees_90} 0 0"/>
                 <geometry>
                     <cylinder radius="${steering_diameter}" length="${steering_width}"/>
                 </geometry>
             </collision>
-            <xacro:default_inertial mass="${steering_mass}"/>
+            <xacro:solid_cylinder_inertial
+                rpy="0 0 0" xyz="0 0 0"
+                mass="${steering_mass}"
+                radius="${steering_diameter/2}" length="${steering_width}" />
         </link>
         <joint name="${prefix}_steering_joint" type="revolute">
@@ -77,5 +84,5 @@
         </joint>
         <!-- The Transmission -->
-        <!-- <transmission name="${prefix}_steering_link_trans">
+        <transmission name="${prefix}_steering_link_trans">
             <type>transmission_interface/SimpleTransmission</type>
             <joint name="${prefix}_steering_joint">
@@ -86,5 +93,5 @@
                 <mechanicalReduction>1</mechanicalReduction>
             </actuator>
-        </transmission> -->
+        </transmission>
     </xacro:macro>
     <!-- Front Wheel Macro -->
@@ -109,29 +116,14 @@
         </link>
         <gazebo reference="${prefix}_front_wheel">
-            <!-- <mu1 value="0.0"/> -->
-            <!-- <mu2 value="0.0"/> -->
-            <!-- <kp value="10000000.0" /> -->
-            <!-- <kd value="1.0" /> -->
             <material>Gazebo/Blue</material>
         </gazebo>
-        <!-- Temporarily join directly to the base_link -->
         <joint name="${prefix}_front_axle" type="continuous">
-            <parent link="base_link"/>
-            <child link="${prefix}_front_wheel"/>
-            <axis xyz="0 1 0"/>
-            <origin xyz="
-                ${body_length / 2 - 0.1}
-                ${(body_width / 2 + steering_width / 2) * reflect + (front_wheel_width/2 + steering_width/2) * reflect}
-                ${-(body_height/2) + 0.1}"
-                rpy="0 0 0"/>
-        </joint>
-        <!-- <joint name="${prefix}_front_axle" type="continuous">
             <parent link="${prefix}_steering_link"/>
             <child link="${prefix}_front_wheel"/>
             <axis xyz="0 1 0"/>
             <origin xyz="0 ${(front_wheel_width/2 + steering_width/2) * reflect} 0"/>
-        </joint> -->
+        </joint>
         <!-- The Transmission -->
-        <!-- <transmission name="${prefix}_front_wheel_trans">
+        <transmission name="${prefix}_front_wheel_trans">
             <type>transmission_interface/SimpleTransmission</type>
             <joint name="${prefix}_front_axle">
@@ -142,13 +134,5 @@
                 <mechanicalReduction>1</mechanicalReduction>
             </actuator>
-        </transmission> -->
-        <gazebo>
-            <plugin name="${prefix}_mimic_joint_plugin" filename="libroboticsgroup_gazebo_mimic_joint_plugin.so">
-                <joint>rear_wheel_joint</joint>
-                <mimicJoint>${prefix}_front_axle</mimicJoint>
-                <multiplier>1</multiplier>
-                <offset>0</offset>
-            </plugin>
-        </gazebo>
+        </transmission>
     </xacro:macro>
     <!-- Rear Wheel Macro -->
@@ -156,5 +140,5 @@
         <link name="${prefix}_rear_wheel">
             <visual>
-                <origin xyz="0.0 0.0 0.0" rpy="${degrees_90} 0.0 0.0"/>
+                <origin xyz="0 0 0" rpy="${degrees_90} 0 0"/>
                 <geometry>
                     <cylinder radius="${rear_wheel_diameter/2}" length="${rear_wheel_width}"/>
@@ -162,5 +146,5 @@
             </visual>
             <collision>
-                <origin xyz="0.0 0.0 0.0" rpy="${degrees_90} 0.0 0.0"/>
+                <origin xyz="0 0 0" rpy="${degrees_90} 0 0"/>
                 <geometry>
                     <cylinder radius="${rear_wheel_diameter/2}" length="${rear_wheel_width}"/>
@@ -173,8 +157,4 @@
         </link>
         <gazebo reference="${prefix}_rear_wheel">
-            <!-- <mu1 value="200.0"/> -->
-            <!-- <mu2 value="100.0"/> -->
-            <!-- <kp value="10000000.0" /> -->
-            <!-- <kd value="1.0" /> -->
             <material>Gazebo/Black</material>
         </gazebo>
@@ -188,11 +168,7 @@
                 ${-(body_height/2) + 0.1}"
                 rpy="0 0 0" />
-            <mimic joint="rear_wheel_joint">
-                <multiplier>1</multiplier>
-                <offset>0</offset>
-            </mimic>
         </joint>
         <!-- The Transmission -->
-        <!-- <transmission name="${prefix}_rear_wheel_trans">
+        <transmission name="${prefix}_rear_wheel_trans">
             <type>transmission_interface/SimpleTransmission</type>
             <joint name="${prefix}_rear_axle">
@@ -203,35 +179,15 @@
                 <mechanicalReduction>1</mechanicalReduction>
             </actuator>
-        </transmission> -->
-        <!-- Mimic joint plugin -->
-        <gazebo>
-            <plugin name="${prefix}_mimic_joint_plugin" filename="libroboticsgroup_gazebo_mimic_joint_plugin.so">
-                <joint>rear_wheel_joint</joint>
-                <mimicJoint>${prefix}_rear_axle</mimicJoint>
-                <!-- if set to true, PID parameters from "/gazebo_ros_control/pid_gains/${mimic_joint}" are loaded -->
-                <!-- <xacro:if value="${has_pid}"> -->
-                <!-- <hasPID /> -->
-                <!-- </xacro:if> -->
-                <multiplier>1</multiplier>
-                <offset>0</offset>
-                <!-- if absolute difference between setpoint and process value is below this threshold, do nothing; 0.0 = disable [rad] -->
-                <!-- <sensitiveness>${sensitiveness}</sensitiveness> -->
-                <!-- only taken into account if has_pid:=true [Nm] -->
-                <!-- <maxEffort>${max_effort}</maxEffort> -->
-                <!-- <xacro:unless value="${robot_namespace == ''}">
-                </xacro:unless>
-                <robotNamespace>($robot_namespace)</robotNamespace> -->
-            </plugin>
-        </gazebo>
+        </transmission>
     </xacro:macro>
-    <!-- <xacro:steering_link prefix="left" reflect="1" /> -->
-    <!-- <xacro:steering_link prefix="right" reflect="-1" /> -->
-    <!-- <xacro:front_wheel_link prefix="left" reflect="1" /> -->
-    <!-- <xacro:front_wheel_link prefix="right" reflect="-1" /> -->
-    <!-- <xacro:rear_wheel_link prefix="left" reflect="1" /> -->
-    <!-- <xacro:rear_wheel_link prefix="right" reflect="-1" /> -->
+    <xacro:steering_link prefix="left" reflect="1" />
+    <xacro:steering_link prefix="right" reflect="-1" />
+    <xacro:front_wheel_link prefix="left" reflect="1" />
+    <xacro:front_wheel_link prefix="right" reflect="-1" />
+    <xacro:rear_wheel_link prefix="left" reflect="1" />
+    <xacro:rear_wheel_link prefix="right" reflect="-1" />
     <link name="front_steer">
         <visual>
-            <origin xyz="0.0 0.0 0.0" rpy="0.0 0.0 0.0"/>
+            <origin xyz="0 0 0" rpy="0 0 0"/>
             <geometry>
                 <cylinder radius="${front_wheel_diameter/2}" length="${front_wheel_width/2}"/>
@@ -239,25 +195,31 @@
         </visual>
         <collision>
-            <origin xyz="0.0 0.0 0.0" rpy="0.0 0.0 0.0"/>
+            <origin xyz="0 0 0" rpy="0 0 0"/>
             <geometry>
                 <cylinder radius="${front_wheel_diameter/2}" length="${front_wheel_width/2}"/>
             </geometry>
         </collision>
-        <xacro:default_inertial mass="${front_wheel_mass}"/>
+        <xacro:solid_cylinder_inertial
+            rpy="${degrees_90} 0 0" xyz="0 0 0"
+            mass="${front_wheel_mass/2}"
+            radius="${front_wheel_diameter/2}" length="${front_wheel_width/2}" />
     </link>
     <link name="rear_wheel">
         <visual>
-            <origin xyz="0.0 0.0 0.0" rpy="${degrees_90} 0.0 0.0"/>
-            <geometry>
-                <cylinder radius="${front_wheel_diameter/2}" length="${front_wheel_width/2}"/>
+            <origin xyz="0 0 0" rpy="${degrees_90} 0 0"/>
+            <geometry>
+                <cylinder radius="${rear_wheel_diameter/2}" length="${rear_wheel_width/2}"/>
             </geometry>
         </visual>
         <collision>
-            <origin xyz="0.0 0.0 0.0" rpy="${degrees_90} 0.0 0.0"/>
-            <geometry>
-                <cylinder radius="${front_wheel_diameter/2}" length="${front_wheel_width/2}"/>
+            <origin xyz="0 0 0" rpy="${degrees_90} 0 0"/>
+            <geometry>
+                <cylinder radius="${rear_wheel_diameter/2}" length="${rear_wheel_width/2}"/>
             </geometry>
         </collision>
-        <xacro:default_inertial mass="${front_wheel_mass}"/>
+        <xacro:solid_cylinder_inertial
+            rpy="${degrees_90} 0 0" xyz="0 0 0"
+            mass="${rear_wheel_mass/2}"
+            radius="${rear_wheel_diameter/2}" length="${rear_wheel_width/2}" />
     </link>
     <joint name="front_steer_joint" type="revolute">
@@ -272,7 +234,6 @@
         <child link="rear_wheel"/>
         <axis xyz="0 1 0"/>
-        <!-- <origin xyz="-0.70 0 " rpy="0 0 0"/> -->
-        <origin xyz="-0.70 0 ${-(body_height/2) - 0.1}" rpy="0 0 0"/>
-        <!-- <limit effort="1000.0" velocity="3.0"/> -->
+        <origin xyz="-0.7 0 0 " rpy="0 0 0"/>
+        <limit effort="1000.0" velocity="3.0"/>
     </joint>
     <transmission name="front_steer_joint_trans">
@@ -296,11 +257,3 @@
         </actuator>
     </transmission>
-    <!-- Gazebo plugin for ROS Control -->
-    <gazebo>
-        <plugin name="gazebo_ros_control" filename="libgazebo_ros_control.so">
-            <robotNamespace>/ursa_bot</robotNamespace>
-            <robotSimType>gazebo_ros_control/DefaultRobotHWSim</robotSimType>
-            <legacyModeNS>false</legacyModeNS>
-        </plugin>
-    </gazebo>
 </robot>
