Commit message: Update bicycle model to use common URDF and refactor.

File: steer_bot_description/urdf/bicycle_bot.urdf.xacro (robot description, xacro)
@@ -14,17 +14,17 @@
     wheel_separation_w = base_width  + 2 * axle_offset = 0.4
 -->
-<robot name="steer_bot" xmlns:xacro="http://wiki.ros.org/xacro">
+<robot name="bicycle_bot" xmlns:xacro="http://wiki.ros.org/xacro">
   <!-- Include xacro for inertials, materials and wheels -->
-  <xacro:include filename="$(find steer_bot_description)/urdf/steer_bot/wheel.xacro"/>
+  <xacro:include filename="$(find steer_bot_description)/urdf/wheel.xacro"/>
   <!-- Math constants -->
   <xacro:property name="deg_to_rad" value="0.01745329251994329577"/>
   <!-- Robot base dimensions -->
   <xacro:property name="base_length" value="0.5" />
-  <xacro:property name="base_width" value="0.3" />
+  <xacro:property name="base_width" value="0.12" />
   <xacro:property name="base_height" value="0.1" />
   <xacro:property name="base_mass" value="5" />
   <!-- Wheel link dimensions -->
   <xacro:property name="wheel_radius" value="0.1" />
-  <xacro:property name="wheel_thickness" value="0.08" />
+  <xacro:property name="wheel_thickness" value="0.1" />
   <xacro:property name="wheel_mass" value="1" />
   <!-- Steering link dimensions -->
@@ -55,5 +55,5 @@
         x="${base_length}" y="${base_width}" z="${base_height}" />
   </link>
-  <!-- Front steer and read wheel joints required for steer_drive_controller -->
+  <!-- Front steer and rear wheel joints required for ackermann_steering_controller -->
   <xacro:front_steer
     name="front"
@@ -71,74 +71,37 @@
     name="rear"
     parent="base"
-    wheel_radius="${wheel_radius/4}"
-    wheel_thickness="${wheel_thickness/2}"
-    wheel_mass="${wheel_mass/32}">
-    <origin xyz="${-base_length/2+axle_offset} 0 0" rpy="${-90 * deg_to_rad} 0 0"/>
-  </xacro:rear_wheel>
-  <!-- Steerable front wheels -->
-  <xacro:front_wheel_lr
-    name="front_right"
-    parent="base"
-    reflect="1"
-    wheel_radius="${wheel_radius}"
-    wheel_thickness="${wheel_thickness}"
-    wheel_mass="${wheel_mass}"
-    steer_radius="${steer_radius}"
-    steer_thickness="${steer_thickness}"
-    steer_mass="${steer_mass}"
-    base_length="${base_length}"
-    base_width="${base_width}"
-    axle_offset="${axle_offset}"
-    steer_height="${wheel_radius+steer_offset}">
-    <origin xyz="${base_length/2-axle_offset} ${base_width/2+axle_offset} 0" rpy="${-90 * deg_to_rad} 0 0"/>
-  </xacro:front_wheel_lr>
-  <xacro:front_wheel_lr
-    name="front_left"
-    parent="base"
-    reflect="-1"
-    wheel_radius="${wheel_radius}"
-    wheel_thickness="${wheel_thickness}"
-    wheel_mass="${wheel_mass}"
-    steer_radius="${steer_radius}"
-    steer_thickness="${steer_thickness}"
-    steer_mass="${steer_mass}"
-    base_length="${base_length}"
-    base_width="${base_width}"
-    axle_offset="${axle_offset}"
-    steer_height="${wheel_radius+steer_offset}">
-    <origin xyz="${base_length/2-axle_offset} ${-base_width/2-axle_offset} 0" rpy="${-90 * deg_to_rad} 0 0"/>
-  </xacro:front_wheel_lr>
-  <!-- Rear wheels -->
-  <xacro:rear_wheel_lr
-    name="rear_right"
-    parent="base"
     wheel_radius="${wheel_radius}"
     wheel_thickness="${wheel_thickness}"
     wheel_mass="${wheel_mass}">
-    <origin xyz="${-base_length/2+axle_offset} ${base_width/2+axle_offset} 0" rpy="${-90 * deg_to_rad} 0 0"/>
-  </xacro:rear_wheel_lr>
-  <xacro:rear_wheel_lr
-    name="rear_left"
-    parent="base"
+    <origin xyz="${-base_length/2+axle_offset} 0 0" rpy="${-90 * deg_to_rad} 0 0"/>
+  </xacro:rear_wheel>
+  <xacro:front_wheel
+    name="front"
+    parent="front_steer"
     wheel_radius="${wheel_radius}"
     wheel_thickness="${wheel_thickness}"
     wheel_mass="${wheel_mass}">
-    <origin xyz="${-base_length/2+axle_offset} ${-base_width/2-axle_offset} 0" rpy="${-90 * deg_to_rad} 0 0"/>
-  </xacro:rear_wheel_lr>
+    <origin xyz="0 0 ${-wheel_radius-steer_offset}" rpy="${-90 * deg_to_rad} 0 0"/>
+  </xacro:front_wheel>
   <!-- Colour -->
   <gazebo reference="base_link">
     <material>Gazebo/Green</material>
   </gazebo>
- <!--
-   Gazebo plugin for ROS Control using the steer_bot_hardware_gazebo
-   implementation of the hardware_interface::RobotHW
- -->
   <gazebo>
+    <!-- Gazebo plugin for ROS Control -->
     <plugin name="gazebo_ros_control" filename="libgazebo_ros_control.so">
       <robotNamespace>/</robotNamespace>
-      <!-- <robotSimType>gazebo_ros_control/DefaultRobotHWSim</robotSimType> -->
-      <robotSimType>steer_bot_hardware_gazebo/SteerBotHardwareGazebo</robotSimType>
+      <robotSimType>gazebo_ros_control/DefaultRobotHWSim</robotSimType>
       <legacyModeNS>false</legacyModeNS>
     </plugin>
   </gazebo>
+  <!-- Load gazebo_ros plugin. Publish passive (non-actuated) joints from Gazebo -->
+  <plugin name="gazebo_ros_joint_state_publisher" filename="libgazebo_ros_joint_state_publisher.so">
+      <robotNamespace>/</robotNamespace>
+      <jointName>
+          front_wheel_joint
+      </jointName>
+      <updateRate>50</updateRate>
+      <alwaysOn>true</alwaysOn>
+  </plugin>
 </robot>

File: steer_bot_description/urdf/wheel.xacro (robot description, xacro)
@@ -9,6 +9,6 @@
 <robot name="wheel" xmlns:xacro="http://wiki.ros.org/xacro">
   <!-- Include xacro for materials and inertials -->
-  <xacro:include filename="$(find steer_bot_description)/urdf/common/materials.xacro"/>
-  <xacro:include filename="$(find steer_bot_description)/urdf/common/inertials.xacro"/>
+  <xacro:include filename="$(find steer_bot_description)/urdf/materials.xacro"/>
+  <xacro:include filename="$(find steer_bot_description)/urdf/inertials.xacro"/>
   <!-- Properties -->
   <xacro:property name="steer_effort" value="10.0"/>
@@ -214,6 +214,6 @@
     </gazebo>
   </xacro:macro>
-  <!-- Car steering model rear wheel links (left/right) -->
-  <xacro:macro name="rear_wheel_lr"
+  <!-- Bicycle model front wheel link (passive - no transmission) -->
+  <xacro:macro name="front_wheel"
     params="
       name
@@ -229,5 +229,5 @@
           <cylinder radius="${wheel_radius}" length="${wheel_thickness}"/>
         </geometry>
-        <material name="red" />
+        <material name="yellow" />
       </visual>
       <collision>
@@ -248,4 +248,42 @@
       <axis xyz="0 0 1"/>
     </joint>
+    <gazebo reference="${name}_wheel_link">
+      <material>Gazebo/Yellow</material>
+    </gazebo>
+  </xacro:macro>
+  <!-- Car steering model rear wheel links (left/right) -->
+  <xacro:macro name="rear_wheel_lr"
+    params="
+      name
+      parent
+      wheel_radius
+      wheel_thickness
+      wheel_mass
+      *origin">
+    <link name="${name}_wheel_link">
+      <visual>
+        <origin xyz="0 0 0" rpy="0 0 0"/>
+        <geometry>
+          <cylinder radius="${wheel_radius}" length="${wheel_thickness}"/>
+        </geometry>
+        <material name="red" />
+      </visual>
+      <collision>
+        <origin xyz="0 0 0" rpy="0 0 0"/>
+        <geometry>
+          <cylinder radius="${wheel_radius}" length="${wheel_thickness}"/>
+        </geometry>
+      </collision>
+      <xacro:solid_cylinder_inertial
+          rpy="0 0 0" xyz="0 0 0"
+          mass="${wheel_mass}"
+          radius="${wheel_radius}" length="${wheel_thickness}" />
+    </link>
+    <joint name="${name}_wheel_joint" type="continuous">
+      <parent link="${parent}_link"/>
+      <child link="${name}_wheel_link"/>
+      <xacro:insert_block name="origin"/>
+      <axis xyz="0 0 1"/>
+    </joint>
     <transmission name="${name}_wheel_joint_trans">
       <type>transmission_interface/SimpleTransmission</type>

Commit message: Fix issue with bicycle model.
1. Fix URDF error where the gazebo plugin element was not enclosed in <gazebo> tags.
2. Fix missing TF for front_wheel_link in rviz.
3. Update namespaces for different models.

File: steer_bot_description/urdf/bicycle_bot.urdf.xacro (robot description, xacro)
@@ -17,4 +17,23 @@
   <!-- Include xacro for inertials, materials and wheels -->
   <xacro:include filename="$(find steer_bot_description)/urdf/wheel.xacro"/>
+  <xacro:property name="robot_namespace" value="/bicycle_bot"/>
+  <!-- Gazebo plugins -->
+  <gazebo>
+    <!-- Load ros_control plugin -->
+    <plugin name="gazebo_ros_control" filename="libgazebo_ros_control.so">
+      <robotNamespace>${robot_namespace}</robotNamespace>
+      <robotSimType>gazebo_ros_control/DefaultRobotHWSim</robotSimType>
+      <legacyModeNS>false</legacyModeNS>
+    </plugin>
+    <!-- Load gazebo_ros plugin. Publish passive (non-actuated) joints from Gazebo -->
+    <plugin name="gazebo_ros_joint_state_publisher" filename="libgazebo_ros_joint_state_publisher.so">
+        <robotNamespace>${robot_namespace}</robotNamespace>
+        <jointName>
+            front_wheel_joint
+        </jointName>
+        <updateRate>50</updateRate>
+        <alwaysOn>true</alwaysOn>
+    </plugin>
+  </gazebo>
   <!-- Math constants -->
   <xacro:property name="deg_to_rad" value="0.01745329251994329577"/>
@@ -68,4 +87,12 @@
     <origin xyz="${base_length/2-axle_offset} 0 0" rpy="${-90 * deg_to_rad} 0 0"/>
   </xacro:front_steer>
+  <xacro:front_wheel
+    name="front"
+    parent="front_steer"
+    wheel_radius="${wheel_radius}"
+    wheel_thickness="${wheel_thickness}"
+    wheel_mass="${wheel_mass}">
+    <origin xyz="0 0 ${-wheel_radius-steer_offset}" rpy="${-90 * deg_to_rad} 0 0"/>
+  </xacro:front_wheel>
   <xacro:rear_wheel
     name="rear"
@@ -76,32 +103,7 @@
     <origin xyz="${-base_length/2+axle_offset} 0 0" rpy="${-90 * deg_to_rad} 0 0"/>
   </xacro:rear_wheel>
-  <xacro:front_wheel
-    name="front"
-    parent="front_steer"
-    wheel_radius="${wheel_radius}"
-    wheel_thickness="${wheel_thickness}"
-    wheel_mass="${wheel_mass}">
-    <origin xyz="0 0 ${-wheel_radius-steer_offset}" rpy="${-90 * deg_to_rad} 0 0"/>
-  </xacro:front_wheel>
   <!-- Colour -->
   <gazebo reference="base_link">
     <material>Gazebo/Green</material>
   </gazebo>
-  <gazebo>
-    <!-- Gazebo plugin for ROS Control -->
-    <plugin name="gazebo_ros_control" filename="libgazebo_ros_control.so">
-      <robotNamespace>/</robotNamespace>
-      <robotSimType>gazebo_ros_control/DefaultRobotHWSim</robotSimType>
-      <legacyModeNS>false</legacyModeNS>
-    </plugin>
-  </gazebo>
-  <!-- Load gazebo_ros plugin. Publish passive (non-actuated) joints from Gazebo -->
-  <plugin name="gazebo_ros_joint_state_publisher" filename="libgazebo_ros_joint_state_publisher.so">
-      <robotNamespace>/</robotNamespace>
-      <jointName>
-          front_wheel_joint
-      </jointName>
-      <updateRate>50</updateRate>
-      <alwaysOn>true</alwaysOn>
-  </plugin>
 </robot>

File: steer_bot_description/urdf/steer_bot.urdf.xacro (robot description, xacro)
@@ -17,4 +17,15 @@
   <!-- Include xacro for inertials, materials and wheels -->
   <xacro:include filename="$(find steer_bot_description)/urdf/wheel.xacro"/>
+  <xacro:property name="robot_namespace" value="/steer_bot"/>
+  <!-- Gazebo plugins -->
+  <gazebo>
+    <!-- Load ros_control plugin using the steer_bot_hardware_gazebo
+    implementation of the hardware_interface::RobotHW -->
+    <plugin name="gazebo_ros_control" filename="libgazebo_ros_control.so">
+      <robotNamespace>${robot_namespace}</robotNamespace>
+      <robotSimType>steer_bot_hardware_gazebo/SteerBotHardwareGazebo</robotSimType>
+      <legacyModeNS>false</legacyModeNS>
+    </plugin>
+  </gazebo>
   <!-- Math constants -->
   <xacro:property name="deg_to_rad" value="0.01745329251994329577"/>
@@ -130,14 +141,3 @@
     <material>Gazebo/Green</material>
   </gazebo>
- <!--
-   Gazebo plugin for ROS Control using the steer_bot_hardware_gazebo
-   implementation of the hardware_interface::RobotHW
-  -->
-  <gazebo>
-    <plugin name="gazebo_ros_control" filename="libgazebo_ros_control.so">
-      <robotNamespace>/</robotNamespace>
-      <robotSimType>steer_bot_hardware_gazebo/SteerBotHardwareGazebo</robotSimType>
-      <legacyModeNS>false</legacyModeNS>
-    </plugin>
-  </gazebo>
 </robot>

File: steer_bot_description/urdf/wheel.xacro (robot description, xacro)
@@ -251,4 +251,7 @@
       <material>Gazebo/Yellow</material>
     </gazebo>
+    <gazebo reference="${name}_wheel_joint">
+      <provideFeedback>true</provideFeedback>
+    </gazebo>
   </xacro:macro>
   <!-- Car steering model rear wheel links (left/right) -->

Commit message: Fix steer_bot has left / right transposed #5
1. Remove unused 'origin' parameters from front wheel and steering macros.
2. Flip signs for reflect and origin-y in steer_bot.

File: steer_bot_description/urdf/bicycle_bot.urdf.xacro (robot description, xacro)
@@ -85,5 +85,4 @@
     axle_offset="${axle_offset}"
     steer_height="${wheel_radius+steer_offset}">
-    <origin xyz="${base_length/2-axle_offset} 0 0" rpy="${-90 * deg_to_rad} 0 0"/>
   </xacro:front_steer>
   <xacro:front_wheel

File: steer_bot_description/urdf/steer_bot.urdf.xacro (robot description, xacro)
@@ -77,5 +77,4 @@
     axle_offset="${axle_offset}"
     steer_height="${wheel_radius+steer_offset}">
-    <origin xyz="${base_length/2-axle_offset} 0 0" rpy="${-90 * deg_to_rad} 0 0"/>
   </xacro:front_steer>
   <xacro:rear_wheel
@@ -91,4 +90,19 @@
     name="front_right"
     parent="base"
+    reflect="-1"
+    wheel_radius="${wheel_radius}"
+    wheel_thickness="${wheel_thickness}"
+    wheel_mass="${wheel_mass}"
+    steer_radius="${steer_radius}"
+    steer_thickness="${steer_thickness}"
+    steer_mass="${steer_mass}"
+    base_length="${base_length}"
+    base_width="${base_width}"
+    axle_offset="${axle_offset}"
+    steer_height="${wheel_radius+steer_offset}">
+  </xacro:front_wheel_lr>
+  <xacro:front_wheel_lr
+    name="front_left"
+    parent="base"
     reflect="1"
     wheel_radius="${wheel_radius}"
@@ -102,21 +116,4 @@
     axle_offset="${axle_offset}"
     steer_height="${wheel_radius+steer_offset}">
-    <origin xyz="${base_length/2-axle_offset} ${base_width/2+axle_offset} 0" rpy="${-90 * deg_to_rad} 0 0"/>
-  </xacro:front_wheel_lr>
-  <xacro:front_wheel_lr
-    name="front_left"
-    parent="base"
-    reflect="-1"
-    wheel_radius="${wheel_radius}"
-    wheel_thickness="${wheel_thickness}"
-    wheel_mass="${wheel_mass}"
-    steer_radius="${steer_radius}"
-    steer_thickness="${steer_thickness}"
-    steer_mass="${steer_mass}"
-    base_length="${base_length}"
-    base_width="${base_width}"
-    axle_offset="${axle_offset}"
-    steer_height="${wheel_radius+steer_offset}">
-    <origin xyz="${base_length/2-axle_offset} ${-base_width/2-axle_offset} 0" rpy="${-90 * deg_to_rad} 0 0"/>
   </xacro:front_wheel_lr>
   <!-- Rear wheels -->
@@ -127,5 +124,5 @@
     wheel_thickness="${wheel_thickness}"
     wheel_mass="${wheel_mass}">
-    <origin xyz="${-base_length/2+axle_offset} ${base_width/2+axle_offset} 0" rpy="${-90 * deg_to_rad} 0 0"/>
+    <origin xyz="${-base_length/2+axle_offset} ${-base_width/2-axle_offset} 0" rpy="${-90 * deg_to_rad} 0 0"/>
   </xacro:rear_wheel_lr>
   <xacro:rear_wheel_lr
@@ -135,5 +132,5 @@
     wheel_thickness="${wheel_thickness}"
     wheel_mass="${wheel_mass}">
-    <origin xyz="${-base_length/2+axle_offset} ${-base_width/2-axle_offset} 0" rpy="${-90 * deg_to_rad} 0 0"/>
+    <origin xyz="${-base_length/2+axle_offset} ${+base_width/2+axle_offset} 0" rpy="${-90 * deg_to_rad} 0 0"/>
   </xacro:rear_wheel_lr>
   <!-- Colour -->

File: steer_bot_description/urdf/wheel.xacro (robot description, xacro)
@@ -25,6 +25,5 @@
       base_width
       axle_offset
-      steer_height
-      *origin">
+      steer_height">
     <link name="${name}_steer_link">
       <visual>
@@ -84,6 +83,5 @@
       base_width
       axle_offset
-      steer_height
-      *origin">
+      steer_height">
     <link name="${name}_steer_link">
       <visual>
